File: Hardware/Radar_Amp/Radar_Amp.kicad_pcb (KiCad board)
At the start: 4 copper layers, 80 x 85 mm, 138 parts, among them J1 Conn_Supply, J2 Conn_Radar, J3 Conn_Output_I, J4 Conn_Output_Q, J5 AudioJack3, U1 OPA_LNA_1, U2 OPA_REF, U3 OPA_LNA_2, U4 OPA_DRIVER, U5 OPA_VGA, U6 OPA_LNA_1, U7 OPA_LNA_2, U8 OPA_VGA, U9 TPS7A20

Commit message: update
Parts:
- moved U9 16.1 mm to (69.6, 69.0)
- moved C26 8.42 mm to (69.6, 64.4)
- moved L2 6.65 mm to (69.6, 57.3)
- moved C45 3.49 mm to (69.6, 50.3)
- moved C27 2.64 mm to (69.6, 73.2)
Connections:
- C26 pad 1: Net-(C26-Pad1) -> Net-(L2-Pad2)
- C26 pad 2: Net-(C26-Pad2) -> GND
- C45 pad 2: Net-(C26-Pad2) -> Net-(C45-Pad2)
- J1 pad 2: Net-(C26-Pad2) -> Net-(C45-Pad2)
- L2 pad 1: Net-(C26-Pad1) -> Net-(C45-Pad1)
- L2 pad 2: +5V -> Net-(L2-Pad2)
- L2 pad 4: Net-(C26-Pad2) -> Net-(C45-Pad2)
- U9 pad 1: Net-(C45-Pad1) -> Net-(L2-Pad2)
- U9 pad 2: Net-(C26-Pad2) -> GND
- U9 pad 3: Net-(C45-Pad1) -> Net-(L2-Pad2)
- U9 pad 5: Net-(C26-Pad1) -> +5V
Routing:
- net Net-(C26-Pad2): track 24.5 -> 0.00 mm
- net Net-(L2-Pad2): track 0.00 -> 11.3 mm
- net Net-(C45-Pad2): track 0.00 -> 10.6 mm
- net Net-(C26-Pad1): track 8.11 -> 0.00 mm
- net GND: track 86.4 -> 90.4 mm, vias 28 -> 29
- net +5V: track 21.3 -> 20.4 mm
- net Net-(C45-Pad1): track 11.2 -> 10.3 mm
