File: Hardware/Radar_Amp/VGA.kicad_sch (KiCad schematic)
At the start: 9 parts, among them U5 OPA_VGA

Commit message: update
Parts:
- renumbered C28 to C44, FB8 to FB11, R26 to R53, R27 to R54, RV1 to RV2, RV3 to RV4, U5 to U8
Changed lines of the file:
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@@
   (symbol (lib_id "Device:Opamp_Dual") (at 194.31 86.36 0)
     (in_bom yes) (on_board yes) (fields_autoplaced)
-    (property "Reference" "U5" (id 0) (at 194.31 76.2 0))
+    (property "Reference" "U8" (id 0) (at 194.31 76.2 0))
     (property "Value" "OPA_VGA" (id 1) (at 194.31 78.74 0))
     (property "Footprint" "Package_SO:SOIC-8_3.9x4.9mm_P1.27mm" (id 2) (at 194.31 86.36 0)
@@
       (effects (font (size 1.27 1.27)) hide)
     )
-    (pin "5")
-    (pin "6")
-    (pin "7")
+    (pin "1")
+    (pin "2")
+    (pin "3")
   )
   (symbol (lib_id "Device:FerriteBead_Small") (at 83.82 30.48 0)
     (in_bom yes) (on_board yes) (fields_autoplaced)
-    (property "Reference" "FB8" (id 0) (at 86.36 29.1718 0)
+    (property "Reference" "FB11" (id 0) (at 86.36 29.1718 0)
       (effects (font (size 1.27 1.27)) (justify left))
     )
@@
   (symbol (lib_id "Device:R_Potentiometer") (at 205.74 100.33 90)
     (in_bom yes) (on_board yes) (fields_autoplaced)
-    (property "Reference" "RV3" (id 0) (at 205.74 104.14 90))
+    (property "Reference" "RV4" (id 0) (at 205.74 104.14 90))
     (property "Value" "R_Potentiometer" (id 1) (at 205.74 106.68 90))
     (property "Footprint" "Potentiometer_SMD:Potentiometer_Bourns_TC33X_Vertical" (id 2) (at 205.74 100.33 0)
@@
   (symbol (lib_id "Device:C_Small") (at 83.82 43.18 0)
     (in_bom yes) (on_board yes) (fields_autoplaced)
-    (property "Reference" "C28" (id 0) (at 86.36 41.9162 0)
+    (property "Reference" "C44" (id 0) (at 86.36 41.9162 0)
       (effects (font (size 1.27 1.27)) (justify left))
     )
@@
   (symbol (lib_id "Device:R") (at 173.99 100.33 90)
     (in_bom yes) (on_board yes) (fields_autoplaced)
-    (property "Reference" "R27" (id 0) (at 173.99 93.98 90))
+    (property "Reference" "R54" (id 0) (at 173.99 93.98 90))
     (property "Value" "300" (id 1) (at 173.99 96.52 90))
     (property "Footprint" "Resistor_SMD:R_1206_3216Metric_Pad1.30x1.75mm_HandSolder" (id 2) (at 173.99 102.108 90)
@@
   (symbol (lib_id "power:GND") (at 83.82 53.34 0)
     (in_bom yes) (on_board yes) (fields_autoplaced)
-    (property "Reference" "#PWR0121" (id 0) (at 83.82 59.69 0)
+    (property "Reference" "#PWR0131" (id 0) (at 83.82 59.69 0)
       (effects (font (size 1.27 1.27)) hide)
     )
@@
   (symbol (lib_id "Device:Opamp_Dual") (at 111.76 86.36 0)
     (in_bom yes) (on_board yes) (fields_autoplaced)
-    (property "Reference" "U5" (id 0) (at 111.76 76.2 0))
+    (property "Reference" "U8" (id 0) (at 111.76 76.2 0))
     (property "Value" "OPA_VGA" (id 1) (at 111.76 78.74 0))
     (property "Footprint" "Package_SO:SOIC-8_3.9x4.9mm_P1.27mm" (id 2) (at 111.76 86.36 0)
@@
   (symbol (lib_id "Device:Opamp_Dual") (at 96.52 43.18 0)
     (in_bom yes) (on_board yes) (fields_autoplaced)
-    (property "Reference" "U5" (id 0) (at 95.25 41.9099 0)
+    (property "Reference" "U8" (id 0) (at 95.25 41.9099 0)
       (effects (font (size 1.27 1.27)) (justify left))
     )
@@
       (effects (font (size 1.27 1.27)) hide)
     )
-    (pin "4")
-    (pin "8")
+    (pin "1")
+    (pin "2")
+    (pin "3")
   )
   (symbol (lib_id "Device:R_Potentiometer") (at 119.38 100.33 90)
     (in_bom yes) (on_board yes) (fields_autoplaced)
-    (property "Reference" "RV1" (id 0) (at 119.38 104.14 90))
+    (property "Reference" "RV2" (id 0) (at 119.38 104.14 90))
     (property "Value" "R_Potentiometer" (id 1) (at 119.38 106.68 90))
     (property "Footprint" "Potentiometer_SMD:Potentiometer_Bourns_TC33X_Vertical" (id 2) (at 119.38 100.33 0)
@@
   (symbol (lib_id "Device:R") (at 93.98 100.33 90)
     (in_bom yes) (on_board yes) (fields_autoplaced)
-    (property "Reference" "R26" (id 0) (at 93.98 93.98 90))
+    (property "Reference" "R53" (id 0) (at 93.98 93.98 90))
     (property "Value" "300" (id 1) (at 93.98 96.52 90))
     (property "Footprint" "Resistor_SMD:R_1206_3216Metric_Pad1.30x1.75mm_HandSolder" (id 2) (at 93.98 102.108 90)
