File: Hardware/Radar_Amp_v2/Radar_Amp_v2.kicad_sch (KiCad schematic)
At the start: 39 parts, among them J1 Conn_Supply, J2 Conn_Radar, U1 TPS7A2033PDBVR, U2 TPS7A2033PDBVR, U3 AD8031

Commit message: fixes
Parts:
- U1, U2: Manufacture # TPS7A2050PDBVR -> TPS7A2033PDBVR
Changed lines of the file:
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@@
       (effects (font (size 1.27 1.27)) hide)
     )
-    (property "Manufacture #" "TPS7A2050PDBVR" (at 95.25 59.69 0)
+    (property "Manufacture #" "TPS7A2033PDBVR" (at 95.25 59.69 0)
       (effects (font (size 1.27 1.27)) hide)
     )
@@
       (effects (font (size 1.27 1.27)) hide)
     )
-    (property "Manufacture #" "TPS7A2050PDBVR" (at 95.25 35.56 0)
-      (effects (font (size 1.27 1.27)) hide)
-    )
+    (property "Manufacture #" "TPS7A2033PDBVR" (at 95.25 35.56 0)
+      (effects (font (size 1.27 1.27)) hide)
+    )
